File: hardware/permamote/rev_b/permamote.brd (EAGLE design)
At the start: 79.4 x 89.5 mm, 137 parts, among them J1 TC2030-JLINK-L, J2 M10X2, J3 M04X2, Q1 PMDXB950UPEL, Q10 CSD22206W, Q11 CSD22206W, Q2 PMDXB950UPEL, Q3 PMDXB950UPEL, Q4 PMDXB950UPEL, Q5 PMDXB950UPEL, Q6 PMDXB950UPEL, Q7 CSD22206W, Q8 CSD22206W, Q9 CSD22206W, U1 AB1815-T3, U10 NRF52840, U11 SI7021-A20-GM1, U2 BQ25505, U3 EKMB1101111, U4 ISL29125, U5 LIS2DW12, U6 MAX17222, U7 MAX44009, U8 MS5637-02BA03, U9 NRF51822QF, X1 32MHz, X2 ABS05-32.768KHZ-9-T, X3 32.768kHz, X4 ABS07-32.768KHZ-7-T, X5 16MHz

Commit message: WIP rev_b
Parts:
- removed A1: ANT3216A063R2400A, chips:ANT3216A063R2400A
- removed B2: BAL-NRF01D3, chips:BAL-NRF01D3
- removed C14, C15: 1nF, passives:0402_CAP
- removed C16: 2.2nF, passives:0402_CAP
- removed C19: 47nF, passives:0402_CAP
- removed C28: 0.1uF, passives:0402_CAP
- removed C3: 0.8pF, passives:0402_CAP
- removed C34: 1uF, passives:0402_CAP
- removed C36: 4.7uF, passives:0402_CAP
- removed C6, C7, C8, C9: 12pF, passives:0402_CAP
- removed H1, H2, H3, H4: MOUNT-PAD-ROUND3.0, holes:3,0-PAD
- removed JP1, JP2, JP3, JP4, JP5, JP6, JP7, JP8: (no value), SparkFun-Passives:SJ_2S
- removed JP10, JP11, JP12, JP13, JP14, JP15, JP16, JP9: (no value), SparkFun-Connectors:1X02
- removed L2: 15nH, passives:0402_CAP
- removed L5: 10uH, passives:0603_CAP
- removed Q11, Q9: CSD22206W, fets:DSBGA
- removed R8: 12kΩ, passives:0402_RES
- removed U9: NRF51822QF, chips:QFN-48-6MM
- removed X2: ABS05-32.768KHZ-9-T, crystals:ABS05
- removed X5: 16MHz, crystals:TXC-8Y
- added C41: 0.1uF, passives:0402_CAP
- added J5: USB-A-MALE_FLARE_LR-PCB, connector:USB-A-MALE_FLARE_LR
- added U12: FT232RQ, ftdichip:QFN32
- Q10, Q7, Q8: value CSD22206W -> PMDXB950UPEL; device fets:DSBGA -> fets:XDFN-6
- R1: value 150Ω -> 10kΩ
- moved R1 203.5 mm to (-58.0, -130.0)
- moved Q8 150.0 mm to (-54.0, -120.0), turned to 0 degrees
- moved Q7 148.9 mm to (-52.0, -115.0), turned to 0 degrees
- moved Q10 148.1 mm to (-56.0, -125.0)
- moved BT2 97.0 mm to (-37.0, 47.0)
- moved BT3 97.0 mm to (-37.0, 24.0)
- moved BT4 97.0 mm to (-37.3, 36.1)
- moved U$1 39.1 mm to (-1.49, 114.9)
Connections:
- removed net AVDD1: C14.1, C34.1, L2.1, U9.35, U9.36
- removed net DCC1: L5.2, U9.2
- removed net N$15: C25.1, C39.1, JP1.1, JP11.1, U5.10, U5.9
- removed net N$19: C26.1, JP15.1, JP4.1, Q9.A2, Q9.A3, Q9.B1, Q9.B2, Q9.B3, R25.2
- removed net N$24: JP14.1, JP8.1, Q11.A2, Q11.A3, Q11.B1, Q11.B2, Q11.B3, R27.2
- removed net N$33: C24.1, C31.1, JP12.1, JP2.1, Q7.A2, Q7.A3, Q7.B1, Q7.B2, Q7.B3, R23.2, R4.2
- removed net N$36: C27.1, JP16.1, JP5.1, Q10.A2, Q10.A3, Q10.B1, Q10.B2, Q10.B3, R26.2
- removed net N$42: C33.1, JP10.1, JP6.1, U1.13
- removed net N$60: B2.ANT1, U9.31
- removed net N$61: B2.ANT2, U9.32
- removed net N$62: A1.S1, B2.SE, C3.1
- removed net N$63: L2.2, L5.1
- removed net N$64: C6.1, U9.37, X5.1
- removed net N$65: C7.1, U9.38, X5.3
- removed net N$66: C15.1, U9.39
- removed net N$67: C19.1, U9.29
- removed net NRF_A2: C9.1, U9.46, X2.B
- removed net NRF_A3: C8.1, U9.45, X2.A
- removed net VCC_JUMP: C20.1, C21.1, C23.1, C28.1, C29.1, C35.1, C36.1, JP7.1, JP9.1, U10.A22, U10.AD14, U10.AD23, U10.B1, U10.W1, U10.Y2, U9.1, U9.12
- removed net VDD_PA1: B2.VCC, C16.1, U9.30
- new net DBG_RX: U12.30
- new net DBG_TX: U12.2
- new net N$13: C41.1, U12.16
- new net USB_5V: J5.+5V, U12.19
- new net USB_D+: J5.D+, U12.14
- new net USB_D-: J5.D-, U12.15
- net !ACC_EN: no longer U10.A14, U9.22
- net !CLR_EN: now also Q7.2; no longer Q7.A1, U9.25
- net !CLR_INT: no longer U9.48
- net !HUM_EN: now also Q8.5; no longer Q10.A1, U9.21
- net !LT_EN: now also Q7.5; no longer Q8.A1, U9.26
- net !LT_INT: no longer U9.47
- net !PIR_EN: now also Q10.2; no longer Q11.A1, U9.27
- net !PR_EN: now also Q8.2; no longer Q9.A1, U9.28
- net !RST: now also U12.18; no longer R1.1
- net !RTC_IRQ1: no longer U9.44
- net !RTC_IRQ2: no longer U9.43
- net !RTC_IRQ3: no longer U9.42
- net ACC_CS: no longer U9.20
- net ACC_INT1: no longer U9.10
- net ACC_INT2: no longer U9.11
- net GND: now also C41.2, J5.GND, U12.17, U12.20, U12.24, U12.26, U12.4; no longer A1.S2, B2.GND, C14.2, C15.2, C16.2, C19.2, C28.2, C3.2, C34.2, C36.2, C6.2, C7.2, C8.2, C9.2, H1.B3,0, H2.B3,0, H3.B3,0, H4.B3,0, R8.2, U9.13, U9.33, U9.34, U9.GND
- net MISO: no longer U9.17
- net MOSI: no longer U9.18
- net N$20: now also Q7.3; no longer Q8.C1, Q8.C2, Q8.C3
- net N$21: now also Q8.6; no longer Q9.C1, Q9.C2, Q9.C3
- net N$22: now also Q8.3; no longer Q10.C1, Q10.C2, Q10.C3
- net N$23: now also Q10.6; no longer Q11.C1, Q11.C2, Q11.C3
- net N$31: now also Q7.6; no longer Q7.C1, Q7.C2, Q7.C3
- net N$37: now also Q7.4; no longer JP13.1, JP3.1, Q8.A2, Q8.A3, Q8.B1, Q8.B2, Q8.B3
- net PIR_OUT: no longer U9.3
- net RTC_CS: no longer U9.41
- net SCK: no longer U9.19
- net SCL: no longer U9.16
- net SDA: no longer U9.14
- net SW: no longer U9.8
- net SWDCLK: no longer R8.1, U9.24
- net SWDIO: no longer J1.6, R1.2, U9.23
- net VBAT: now also C33.1, R1.2, U1.13; no longer JP10.2, JP6.2, U9.6
- net VCC: now also C20.1, C21.1, C23.1, C24.1, C25.1, C26.1, C27.1, C29.1, C31.1, C35.1, C39.1, Q10.1, Q7.1, Q8.1, Q8.4, R23.2, R25.2, R26.2, R27.2, R4.2, U10.A22, U10.AD14, U10.AD23, U10.B1, U10.W1, U10.Y2, U12.1, U5.10, U5.9; no longer JP1.2, JP11.2, JP12.2, JP13.2, JP14.2, JP15.2, JP16.2, JP2.2, JP3.2, JP4.2, JP5.2, JP7.2, JP8.2, JP9.2
- net VSEC: no longer U9.5
- net VSOL: no longer U9.7
- net WDI: now also R1.1; no longer U9.40
Routing:
- net VBAT: track 219.8 -> 0.00 mm, vias 5 -> 0
- net SCL: track 187.9 -> 0.00 mm, vias 10 -> 0
- net SDA: track 181.7 -> 0.00 mm, vias 9 -> 0
- net !LT_INT: track 169.0 -> 0.00 mm, vias 7 -> 0
- net !HUM_EN: track 164.7 -> 0.00 mm, vias 7 -> 0
- net MOSI: track 164.5 -> 0.00 mm, vias 6 -> 0
- net !CLR_EN: track 162.7 -> 0.00 mm, vias 8 -> 0
- net MISO: track 161.8 -> 0.00 mm, vias 6 -> 0
- net !CLR_INT: track 160.5 -> 0.00 mm, vias 7 -> 0
- net !RST: track 160.4 -> 0.00 mm, vias 5 -> 0
- net SCK: track 155.9 -> 0.00 mm, vias 6 -> 0
- net VSOL: track 155.2 -> 0.00 mm, vias 5 -> 0
- net !PR_EN: track 144.1 -> 0.00 mm, vias 6 -> 0
- net !LT_EN: track 143.7 -> 0.00 mm, vias 7 -> 0
- net ACC_INT2: track 139.1 -> 0.00 mm, vias 5 -> 0
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- removed copper zone on layer 15, net N$38
- removed copper zone on layer 16, net N$38
- removed copper zone on layer 2, net N$38
Other:
- board size 79.4 x 89.5 mm -> 79.4 x 89 mm
- board text removed: "2/3 AA"
- board text removed: "AA"
- board text removed: "CR123A"
- board text removed: "NRF51822"
