File: hardware/permamote/rev_b/permamote.sch (EAGLE design)
At the start: 136 parts, among them J1 TC2030-JLINK-L, J2 M10X2, J3 M04X2, Q1 PMDXB950UPEL, Q10 CSD22206W, Q11 CSD22206W, Q2 PMDXB950UPEL, Q3 PMDXB950UPEL, Q4 PMDXB950UPEL, Q5 PMDXB950UPEL, Q6 PMDXB950UPEL, Q7 CSD22206W, Q8 CSD22206W, Q9 CSD22206W, U1 AB1815-T3, U10 NRF52840, U11 SI7021-A20-GM1, U2 BQ25505, U3 EKMB1101111, U4 ISL29125, U5 LIS2DW12, U6 MAX17222, U7 MAX44009, U8 MS5637-02BA03, U9 NRF51822QF, X1 32MHz, X2 ABS05-32.768KHZ-9-T, X3 32.768kHz, X4 ABS07-32.768KHZ-7-T, X5 16MHz

Commit message: WIP rev_b
Parts:
- removed A1: ANT3216A063R2400A, chips:ANT3216A063R2400A
- removed B2: BAL-NRF01D3, chips:BAL-NRF01D3
- removed C14, C15: 1nF, passives:CAPACITOR0402_CAP
- removed C16: 2.2nF, passives:CAPACITOR0402_CAP
- removed C19: 47nF, passives:CAPACITOR0402_CAP
- removed C28: 0.1uF, passives:CAPACITOR0402_CAP
- removed C3: 0.8pF, passives:CAPACITOR0402_CAP
- removed C34: 1uF, passives:CAPACITOR0402_CAP
- removed C36: 4.7uF, passives:CAPACITOR0402_CAP
- removed C6, C7, C8, C9: 12pF, passives:CAPACITOR0402_CAP
- removed H1, H2, H3, H4: MOUNT-PAD-ROUND3.0, holes:MOUNT-PAD-ROUND3.0
- removed JP1, JP2, JP3, JP4, JP5, JP6, JP7, JP8: (no value), SparkFun-Passives:JUMPER-2SMD-NC
- removed JP10, JP11, JP12, JP13, JP14, JP15, JP16, JP9: (no value), SparkFun-Connectors:M02PTH
- removed L2: 15nH, passives:INDUCTOR0402
- removed L5: 10uH, passives:INDUCTOR0603
- removed Q11, Q9: CSD22206W, fets:CSD22206W
- removed R8: 12kΩ, passives:RESISTOR0402_RES
- removed U9: NRF51822QF, chips:NRF51822QF
- removed X2: ABS05-32.768KHZ-9-T, crystals:ABS05-32.768KHZ-9-T
- removed X5: 16MHz, crystals:TXC-8Y
- added C41: 0.1uF, passives:CAPACITOR0402_CAP
- added J5: USB-A-MALE_FLARE_LR-PCB, connector:USB-A-MALE_FLARE_LR-PCB
- added U12: FT232RQ, ftdichip:FT232RQ
- Q10, Q7, Q8: value CSD22206W -> PMDXB950UPEL; device fets:CSD22206W -> fets:PMDXB950UPEL
- R1: value 150Ω -> 10kΩ; DIGIKEY 311-150JRCT-ND -> 311-10KJRCT-ND
Connections:
- removed net AVDD1: C14.1, C34.1, L2.1, U9.AVDD
- removed net DCC1: L5.2, U9.DCC
- removed net N$15: C25.1, C39.1, JP1.1, JP11.1, U5.VCC, U5.VDD_IO
- removed net N$19: C26.1, JP15.1, JP4.1, Q9.S, R25.2
- removed net N$24: JP14.1, JP8.1, Q11.S, R27.2
- removed net N$33: C24.1, C31.1, JP12.1, JP2.1, Q7.S, R23.2, R4.2
- removed net N$36: C27.1, JP16.1, JP5.1, Q10.S, R26.2
- removed net N$42: C33.1, JP10.1, JP6.1, U1.VCC
- removed net N$60: B2.ANT1, U9.ANT1
- removed net N$61: B2.ANT2, U9.ANT2
- removed net N$62: A1.ANTENNA, B2.SE, C3.1
- removed net N$63: L2.2, L5.1
- removed net N$64: C6.1, U9.XC1, X5.1
- removed net N$65: C7.1, U9.XC2, X5.2
- removed net N$66: C15.1, U9.DEC1
- removed net N$67: C19.1, U9.DEC2
- removed net NRF_A2: C9.1, U9.P27/AIN1/XL1, X2.2
- removed net NRF_A3: C8.1, U9.P26/AIN0/XL2, X2.1
- removed net VCC_JUMP: C20.1, C21.1, C23.1, C28.1, C29.1, C35.1, C36.1, JP7.1, JP9.1, U10.VDD, U10.VDDH, U9.VDD
- removed net VDD_PA1: B2.VDD_PA, C16.1, U9.VDD_PA
- new net DBG_RX: U12.TXD
- new net DBG_TX: U12.RXD
- new net N$13: C41.1, U12.3V3OUT
- new net USB_5V: J5.+5V, U12.VCC
- new net USB_D+: J5.D+, U12.USBDP
- new net USB_D-: J5.D-, U12.USBDM
- net !ACC_EN: no longer U10.P1.15, U9.P16
- net !CLR_EN: now also Q7.1.G; no longer Q7.G, U9.P17
- net !CLR_INT: no longer U9.P29
- net !HUM_EN: now also Q8.2.G; no longer Q10.G, U9.P15
- net !LT_EN: now also Q7.2.G; no longer Q8.G, U9.P18
- net !LT_INT: no longer U9.P28
- net !PIR_EN: now also Q10.1.G; no longer Q11.G, U9.P19
- net !PR_EN: now also Q8.1.G; no longer Q9.G, U9.P20
- net !RST: now also U12.!RESET; no longer R1.1
- net !RTC_IRQ1: no longer U9.P25
- net !RTC_IRQ2: no longer U9.P24
- net !RTC_IRQ3: no longer U9.P23
- net ACC_CS: no longer U9.P14
- net ACC_INT1: no longer U9.P06/AIN7/AREF1
- net ACC_INT2: no longer U9.P07
- net GND: now also C41.2, J5.GND, U12.GND, U12.GND@1, U12.GND@2, U12.GND@A, U12.TEST; no longer A1.GND, B2.GND, C14.2, C15.2, C16.2, C19.2, C28.2, C3.2, C34.2, C36.2, C6.2, C7.2, C8.2, C9.2, H1.MOUNT, H2.MOUNT, H3.MOUNT, H4.MOUNT, R8.2, U9.GND
- net MISO: no longer U9.P11
- net MOSI: no longer U9.P12
- net N$20: now also Q7.2.D; no longer Q8.D
- net N$21: now also Q8.1.D; no longer Q9.D
- net N$22: now also Q8.2.D; no longer Q10.D
- net N$23: now also Q10.1.D; no longer Q11.D
- net N$31: now also Q7.1.D; no longer Q7.D
- net N$37: now also Q7.2.S; no longer JP13.1, JP3.1, Q8.S
- net PIR_OUT: no longer U9.P30
- net RTC_CS: no longer U9.P22
- net SCK: no longer U9.P13
- net SCL: no longer U9.P10
- net SDA: no longer U9.P08
- net SW: no longer U9.P04/AIN5
- net SWDCLK: no longer R8.1, U9.SWDCLK
- net SWDIO: no longer J1.SWO, R1.2, U9.SWDIO/!RESET
- net VBAT: now also C33.1, R1.2, U1.VCC; no longer JP10.2, JP6.2, U9.P02/AIN3
- net VCC: now also C20.1, C21.1, C23.1, C24.1, C25.1, C26.1, C27.1, C29.1, C31.1, C35.1, C39.1, Q10.1.S, Q7.1.S, Q8.1.S, Q8.2.S, R23.2, R25.2, R26.2, R27.2, R4.2, U10.VDD, U10.VDDH, U12.VCCIO, U5.VCC, U5.VDD_IO; no longer JP1.2, JP11.2, JP12.2, JP13.2, JP14.2, JP15.2, JP16.2, JP2.2, JP3.2, JP4.2, JP5.2, JP7.2, JP8.2, JP9.2
- net VSEC: no longer U9.P01/AIN2
- net VSOL: no longer U9.P03/AIN4
- net WDI: now also R1.1; no longer U9.P21
Other:
- note added: "Debugging"
- note removed: "Auxillary NRF51822"
- note removed: "Mounting Holes"
